Commit message: Add new file

File: src/robot_description_description/urdf/materials.xacro (robot description, xacro)
@@ -1,6 +1,12 @@
 <?xml version="1.0" ?>
-<robot name="robot_description" xmlns:xacro="http://www.ros.org/wiki/xacro" >
+<robot name="diff_robot" xmlns:xacro="http://www.ros.org/wiki/xacro" >
 <material name="silver">
   <color rgba="0.700 0.700 0.700 1.000"/>
 </material>
+<material name="blue">
+  <color rgba="0.400 0.300 1.000 1.000"/>
+</material>
+<material name="orange">
+  <color rgba="0.900 0.500 0.300 1.000"/>
+</material>
 </robot>

File: src/robot_description_description/urdf/robot_description.xacro (robot description, xacro)
@@ -1,7 +1,14 @@
 <?xml version="1.0" ?>
-<robot name="robot_description" xmlns:xacro="http://www.ros.org/wiki/xacro">
+<robot name="diff_robot" xmlns:xacro="http://www.ros.org/wiki/xacro">
+<!-- materials file -->
 <xacro:include filename="$(find robot_description_description)/urdf/materials.xacro" />
-<xacro:include filename="$(find robot_description_description)/urdf/robot_description.trans" />
-<xacro:include filename="$(find robot_description_description)/urdf/robot_description.gazebo" />
+<!-- gazebo materials file -->
+<xacro:include filename="$(find robot_description_description)/gazebo/robot_description_gazebo_material.gazebo" />
+<!-- transfer -->
+<!-- <xacro:include filename="$(find robot_description_description)/urdf/robot_description.trans" /> -->
+<!-- plugin -->
+<xacro:include filename="$(find robot_description_description)/gazebo/robot_description_gazebo_plugin.gazebo" />
+<xacro:include filename="$(find robot_description_description)/gazebo/robot_description.gazebo" />
+<!-- link -->
 <link name="base_link">
   <inertial>
@@ -15,5 +22,5 @@
       <mesh filename="package://robot_description_description/meshes/base_link.stl" scale="0.001 0.001 0.001"/>
     </geometry>
-    <material name="silver"/>
+    <material name="blue"/>
   </visual>
   <collision>
@@ -35,5 +42,5 @@
       <mesh filename="package://robot_description_description/meshes/lidar_1.stl" scale="0.001 0.001 0.001"/>
     </geometry>
-    <material name="silver"/>
+    <material name="blue"/>
   </visual>
   <collision>
@@ -55,5 +62,5 @@
       <mesh filename="package://robot_description_description/meshes/left_wheel_1.stl" scale="0.001 0.001 0.001"/>
     </geometry>
-    <material name="silver"/>
+    <material name="orange"/>
   </visual>
   <collision>
@@ -75,5 +82,5 @@
       <mesh filename="package://robot_description_description/meshes/right_wheel_1.stl" scale="0.001 0.001 0.001"/>
     </geometry>
-    <material name="silver"/>
+    <material name="orange"/>
   </visual>
   <collision>
@@ -84,10 +91,11 @@
   </collision>
 </link>
-<joint name="Rigid10" type="fixed">
+<!-- joint -->
+<joint name="to_lidar" type="fixed">
   <origin xyz="-0.09 0.0 0.141" rpy="0 0 0"/>
   <parent link="base_link"/>
   <child link="lidar_1"/>
 </joint>
-<joint name="Rev11" type="continuous">
+<joint name="to_left_wheel" type="continuous">
   <origin xyz="-0.1 0.097 0.035" rpy="0 0 0"/>
   <parent link="base_link"/>
@@ -95,5 +103,5 @@
   <axis xyz="0.0 1.0 0.0"/>
 </joint>
-<joint name="Rev12" type="continuous">
+<joint name="to_right_wheel" type="continuous">
   <origin xyz="-0.1 -0.097 0.035" rpy="0 0 0"/>
   <parent link="base_link"/>
